Commit message: Fixed a few model issues, launch file, and map settings

File: brain/src/chuck_model/urdf/chuck.urdf.xacro (robot description, xacro)
@@ -7,5 +7,22 @@
 	<xacro:include filename="$(find chuck_model)/urdf/component/caster.urdf.xacro"/>
 	<!-- Robot footprint -->
-	<link name="base_footprint"/>
+	<link name="base_footprint">
+	    <inertial>
+	      <mass value="0.0001" />
+	      <origin xyz="0 0 0" />
+	      <inertia ixx="0.0001" ixy="0.0" ixz="0.0"
+	          iyy="0.0001" iyz="0.0"
+	          izz="0.0001" />
+	    </inertial>
+	    <visual>
+	        <origin xyz="0 0 0" rpy="0 0 0" />
+	        <geometry>
+	            <box size="0.001 0.001 0.001" />
+	        </geometry>
+	    </visual>
+    </link>
+	<gazebo reference="base_footprint">
+		<turnGravityOff>false</turnGravityOff>
+	</gazebo>
 	<joint name="base_footprint_joint" type="fixed">
 		<origin xyz="0 0 0" rpy="0 0 0"/>
@@ -56,8 +73,8 @@
 	</link>
 	<!-- Wheels -->
-	<wheel lr="left" parent="base_link" side="1"/>
-	<wheel lr="right" parent="base_link" side="-1"/>
+	<wheel lr="left" parent="base_link" translateX="0" translateY="${-base_x_size/2}" translateZ="0" />
+	<wheel lr="right" parent="base_link" translateX="0"  translateY="${base_x_size/2}" translateZ="0" />
 	<!-- Castors -->
-	<castor fb="front" parent="base_link" side="-1"/>
-	<castor fb="back" parent="base_link" side="-1"/>
+	<castor fb="front" parent="base_link" translateX="1" translateY="0" translateZ="0" />
+	<castor fb="back" parent="base_link" translateX="-1" translateY="0" translateZ="0" />
 </robot>

File: brain/src/chuck_model/urdf/component/caster.urdf.xacro (robot description, xacro)
@@ -2,8 +2,8 @@
 <robot name="caster" xmlns:xacro="http://www.ros.org/wiki/xacro">
 	<xacro:include filename="$(find chuck_model)/urdf/common/inertia.xacro"/>
-	<xacro:macro name="caster" params="fb parent side">
+	<xacro:macro name="caster" params="fb parent translateX translateY translateZ">
 	    <link name="${fb}_caster_body">
             <visual>
-                <origin xyz="0 0 0" rpy="0 0 0"/>
+				<origin xyz="0 0 0" rpy="${M_PI/2} 0  0 " />
                 <geometry>
                     <box size="${caster_x_size} ${caster_y_size} ${caster_z_size}"/>
@@ -12,5 +12,5 @@
             </visual>
             <collision>
-                <origin xyz="0 0 0" rpy="0 0 0 " />
+				<origin xyz="0 0 0" rpy="${M_PI/2} 0  0 " />
                 <geometry>
                     <box size="${caster_x_size} ${caster_y_size} ${caster_z_size}"/>
@@ -26,5 +26,5 @@
             <parent link="${parent}"/>
             <child link="${fb}_caster_body"/>
-            <origin xyz="${side * (base_x_size / 2 + 0.05)} 0 0" rpy="0 0 0"/>
+			<origin xyz="${translateX} ${translateY} ${translateZ}" rpy="0 0 0"/>
             <axis xyz="0 1 0" rpy="0 0 0" />
         </joint>

File: brain/src/chuck_model/urdf/component/wheel.urdf.xacro (robot description, xacro)
@@ -2,8 +2,8 @@
 <robot name="wheel" xmlns:xacro="http://www.ros.org/wiki/xacro">
 	<xacro:include filename="$(find chuck_model)/urdf/common/inertia.xacro"/>
-	<xacro:macro name="wheel" params="lr parent side">
+	<xacro:macro name="wheel" params="lr parent translateX translateY translateZ">
 		<link name="${lr}_wheel">
 			<visual>
-				<origin xyz="0 0 ${base_offset}" rpy="${-M_PI/2} 0 0"/>
+				<origin xyz="0 0 0" rpy="${M_PI/2} 0  0 " />
 				<geometry>
 					<cylinder length="${wheel_thickness}" radius="${wheel_radius}"/>
@@ -12,5 +12,5 @@
 			</visual>
 			<collision>
-				<origin xyz="0 0 ${base_offset}" rpy="${-M_PI/2} 0 0"/>
+				<origin xyz="0 0 0" rpy="${M_PI/2} 0 0 " />
 				<geometry>
 					<cylinder length="${wheel_thickness}" radius="${wheel_radius}"/>
@@ -26,5 +26,5 @@
 			<parent link="${parent}"/>
 			<child link="${lr}_wheel"/>
-			<origin xyz="0 ${side * (base_z_size + wheel_thickness / 2 + 0.01)} ${body_zero - base_z_size / 2}" rpy="0 0 0"/>
+			<origin xyz="${translateX} ${translateY} ${translateZ}" rpy="0 0 0"/>
 			<axis xyz="0 1 0" rpy="0 0 0"/>
 			<limit effort="100" velocity="100"/>

File: brain/src/chuck_model/urdf/properties.xacro (robot description, xacro)
@@ -3,4 +3,6 @@
 	<!-- All units in m-kg-s-radians unit system -->
 	<xacro:property name="M_PI" value="3.1415926535897931"/>
+	<xacro:property name="M_PI_2" value="1.570796327" />
+	<xacro:property name="DEG_TO_RAD" value="0.017453293" />
 	<!-- Chassis -->
 	<xacro:property name="base_x_size" value="0.787"/>
@@ -26,8 +28,8 @@
 	<xacro:property name="tray_zero" value="${support_zero + support_z_size / 2 + tray_z_size / 2}"/>
 	<!-- Wheels -->
-	<xacro:property name="wheel_radius" value="0.100"/>
+	<xacro:property name="wheel_radius" value="0.12500"/>
 	<xacro:property name="wheel_thickness" value="0.050"/>
 	<xacro:property name="wheel_mass" value="2.5"/>
-	<xacro:property name="caster_radius" value="0.050"/>
+	<xacro:property name="caster_radius" value="0.200"/>
 	<xacro:property name="caster_thickness" value="0.025"/>
 	<xacro:property name="caster_mass" value="3.0"/>
@@ -35,4 +37,3 @@
 	<xacro:property name="caster_y_size" value="0.1"/>
 	<xacro:property name="caster_z_size" value="0.2"/>
-	<xacro:property name="caster_offset" value="-0.111"/>
 </robot>

Commit message: Fixed castor URDF

File: brain/src/chuck_model/urdf/chuck.urdf.xacro (robot description, xacro)
@@ -73,8 +73,8 @@
 	</link>
 	<!-- Wheels -->
-	<wheel lr="left" parent="base_link" translateX="0" translateY="${-base_x_size/2}" translateZ="0" />
-	<wheel lr="right" parent="base_link" translateX="0"  translateY="${base_x_size/2}" translateZ="0" />
+	<wheel lr="left" parent="base_link" translateX="0" translateY="${-wheel_y_offset}" translateZ="0" />
+	<wheel lr="right" parent="base_link" translateX="0"  translateY="${wheel_y_offset}" translateZ="0" />
 	<!-- Castors -->
-	<castor fb="front" parent="base_link" translateX="1" translateY="0" translateZ="0" />
-	<castor fb="back" parent="base_link" translateX="-1" translateY="0" translateZ="0" />
+	<caster fb="front" parent="base_link" translateX="${caster_front_x_offset}" translateY="0" translateZ="${caster_z_offset}" />
+	<caster fb="back" parent="base_link" translateX="${caster_back_x_offset}" translateY="0" translateZ="${caster_z_offset}" />
 </robot>

File: brain/src/chuck_model/urdf/component/caster.urdf.xacro (robot description, xacro)
@@ -5,5 +5,5 @@
 	    <link name="${fb}_caster_body">
             <visual>
-				<origin xyz="0 0 0" rpy="${M_PI/2} 0  0 " />
+				<origin xyz="0 0 0" rpy="0 0 0" />
                 <geometry>
                     <box size="${caster_x_size} ${caster_y_size} ${caster_z_size}"/>
@@ -12,5 +12,5 @@
             </visual>
             <collision>
-				<origin xyz="0 0 0" rpy="${M_PI/2} 0  0 " />
+				<origin xyz="0 0 0" rpy="0 0 0" />
                 <geometry>
                     <box size="${caster_x_size} ${caster_y_size} ${caster_z_size}"/>
@@ -23,5 +23,5 @@
             </inertial>
         </link>
-        <joint name="joint_front_caster_body" type="fixed">
+        <joint name="joint_${fb}_caster_body" type="continuous">
             <parent link="${parent}"/>
             <child link="${fb}_caster_body"/>
@@ -31,4 +31,5 @@
         <link name="${fb}_caster_wheel">
             <visual>
+				<origin xyz="0 0 0" rpy="${M_PI/2} 0  0 " />
                 <geometry>
                     <cylinder length="${caster_thickness}" radius="${caster_radius}"/>
@@ -37,4 +38,5 @@
             </visual>
             <collision>
+				<origin xyz="0 0 0" rpy="${M_PI/2} 0  0 " />
                 <geometry>
                     <cylinder length="${caster_thickness}" radius="${caster_radius}"/>
@@ -47,8 +49,10 @@
         </link>
         <joint name="${fb}_caster_wheel_joint" type="continuous">
-            <axis xyz="0 0 1"/>
             <parent link="${fb}_caster_body"/>
             <child link="${fb}_caster_wheel"/>
-            <origin rpy="-1.5708 0 0" xyz="${side * 0.05} 0 ${caster_offset}"/>
+			<origin xyz="0 0 0" rpy="0 0 0"/>
+			<axis xyz="0 1 0" rpy="0 0 0"/>
+			<limit effort="100" velocity="100"/>
+			<joint_properties damping="0.0" friction="0.0"/>
         </joint>
 		<gazebo reference="${fb}_caster">

File: brain/src/chuck_model/urdf/properties.xacro (robot description, xacro)
@@ -6,9 +6,9 @@
 	<xacro:property name="DEG_TO_RAD" value="0.017453293" />
 	<!-- Chassis -->
-	<xacro:property name="base_x_size" value="0.787"/>
-	<xacro:property name="base_y_size" value="0.647"/>
-	<xacro:property name="base_z_size" value="0.266"/>
+	<xacro:property name="base_x_size" value="0.9772396"/>
+	<xacro:property name="base_y_size" value="0.619125"/>
+	<xacro:property name="base_z_size" value="0.3010916"/>
 	<xacro:property name="base_offset" value="0.070"/>
-	<xacro:property name="base_mass" value="90."/>
+	<xacro:property name="base_mass" value="4.53592"/>
 	<!-- Tray support -->
 	<xacro:property name="support_x_size" value="0.050"/>
@@ -28,8 +28,10 @@
 	<xacro:property name="tray_zero" value="${support_zero + support_z_size / 2 + tray_z_size / 2}"/>
 	<!-- Wheels -->
-	<xacro:property name="wheel_radius" value="0.12500"/>
-	<xacro:property name="wheel_thickness" value="0.050"/>
-	<xacro:property name="wheel_mass" value="2.5"/>
-	<xacro:property name="caster_radius" value="0.200"/>
+	<xacro:property name="wheel_radius" value="0.2032"/>
+	<xacro:property name="wheel_thickness" value="0.047625"/>
+	<xacro:property name="wheel_mass" value="2.118276"/>
+	<xacro:property name="wheel_y_offset" value="0.2661285"/>
+	<xacro:property name="wheel_z_offset" value="0"/>
+	<xacro:property name="caster_radius" value="0.100"/>
 	<xacro:property name="caster_thickness" value="0.025"/>
 	<xacro:property name="caster_mass" value="3.0"/>
@@ -37,3 +39,6 @@
 	<xacro:property name="caster_y_size" value="0.1"/>
 	<xacro:property name="caster_z_size" value="0.2"/>
+	<xacro:property name="caster_front_x_offset" value="0.2885948"/>
+	<xacro:property name="caster_back_x_offset" value="-0.3564382"/>
+	<xacro:property name="caster_z_offset" value="${caster_y_size - wheel_radius}"/>
 </robot>

Commit message: model changes

File: brain/src/chuck_model/urdf/chuck.urdf.xacro (robot description, xacro)
@@ -75,3 +75,4 @@
 	<caster fb="front" parent="base_link" translateX="${caster_front_x_offset}" translateY="0" translateZ="${caster_z_offset}" />
 	<caster fb="back" parent="base_link" translateX="${caster_back_x_offset}" translateY="0" translateZ="${caster_z_offset}" />
+	<xacro:include filename="$(find chuck_model)/urdf/chuck.gazebo"/>
 </robot>

File: brain/src/chuck_model/urdf/component/caster.urdf.xacro (robot description, xacro)
@@ -3,64 +3,32 @@
 	<xacro:include filename="$(find chuck_model)/urdf/common/inertia.xacro"/>
 	<xacro:macro name="caster" params="fb parent translateX translateY translateZ">
-	    <link name="${fb}_caster_body">
-            <visual>
-				<origin xyz="0 0 0" rpy="0 0 0" />
-                <geometry>
-                    <box size="${caster_x_size} ${caster_y_size} ${caster_z_size}"/>
-                </geometry>
-                <material name="DarkGray"/>
-            </visual>
-            <collision>
-				<origin xyz="0 0 0" rpy="0 0 0" />
-                <geometry>
-                    <box size="${caster_x_size} ${caster_y_size} ${caster_z_size}"/>
-                </geometry>
-            </collision>
-            <inertial>
-                <mass value="1" />
-                <origin xyz="0 0 0" />
-                <box_inertia m="1" x="${caster_x_size}" y="${caster_y_size}" z="${caster_z_size}"/>
-            </inertial>
-        </link>
-        <joint name="joint_${fb}_caster_body" type="continuous">
-            <parent link="${parent}"/>
-            <child link="${fb}_caster_body"/>
-			<origin xyz="${translateX} ${translateY} ${translateZ}" rpy="0 0 0"/>
-            <axis xyz="0 1 0" rpy="0 0 0" />
-        </joint>
-        <link name="${fb}_caster_wheel">
-            <visual>
-				<origin xyz="0 0 0" rpy="${M_PI/2} 0  0 " />
-                <geometry>
-                    <cylinder length="${caster_thickness}" radius="${caster_radius}"/>
-                </geometry>
-                <material name="black"/>
-            </visual>
-            <collision>
-				<origin xyz="0 0 0" rpy="${M_PI/2} 0  0 " />
-                <geometry>
-                    <cylinder length="${caster_thickness}" radius="${caster_radius}"/>
-                </geometry>
-            </collision>
-            <inertial>
-                <mass value="1"/>
-                <cylinder_inertia m="${caster_mass}" r="${caster_radius}" h="${caster_thickness}"/>
-            </inertial>
-        </link>
-        <joint name="${fb}_caster_wheel_joint" type="continuous">
-            <parent link="${fb}_caster_body"/>
-            <child link="${fb}_caster_wheel"/>
-			<origin xyz="0 0 0" rpy="0 0 0"/>
-			<axis xyz="0 1 0" rpy="0 0 0"/>
-			<limit effort="100" velocity="100"/>
-			<joint_properties damping="0.0" friction="0.0"/>
-        </joint>
-		<gazebo reference="${fb}_caster">
-			<mu1 value="1.0"/>
-			<mu2 value="1.0"/>
-			<kp  value="10000000.0"/>
-			<kd  value="1.0"/>
-			<fdir1 value="1 0 0"/>
-			<material>Gazebo/Grey</material>
+	    <link name="${fb}_caster">
+			<visual>
+				<origin xyz="0 0.02 0" rpy="${M_PI/2} 0 0" />
+				<geometry>
+					<sphere radius="${caster_radius}" />
+				</geometry>
+				<material name="Black" />
+			</visual>
+			<collision>
+				<origin xyz="0 0 0" rpy="${M_PI/2} 0 0" />
+				<geometry>
+					<sphere radius="${caster_radius}" />
+				</geometry>
+			</collision>
+			<inertial>
+				<mass value="${caster_mass}" />
+				<origin xyz="0 0 0" />
+				<inertia ixx="0.001" ixy="0.0" ixz="0.0"
+	                 iyy="0.001" iyz="0.0"
+	                 izz="0.001" />
+			</inertial>
+		</link>
+		<joint name="caster_${fb}_joint" type="fixed">
+			<parent link="${parent}"/>
+			<child link="${fb}_caster"/>
+			<origin xyz="${translateX} ${translateY} ${translateZ}" rpy="${-M_PI/2} 0 0"/>
+		</joint>
+		<gazebo reference="caster_${fb}_link">
 			<turnGravityOff>false</turnGravityOff>
 		</gazebo>

File: brain/src/chuck_model/urdf/component/wheel.urdf.xacro (robot description, xacro)
@@ -34,5 +34,7 @@
 		<transmission name="${lr}_wheel_joint_trans">
 			<type>transmission_interface/SimpleTransmission</type>
-			<joint name="${lr}_wheel_joint"/>
+			<joint name="${lr}_wheel_joint" >
+				<hardwareInterface>EffortJointInterface</hardwareInterface>
+			</joint>
 			<actuator name="${lr}_wheel_joint_motor">
 				<hardwareInterface>EffortJointInterface</hardwareInterface>

Commit message: Fixed issues with model and launch files

File: brain/src/chuck_model/urdf/chuck.urdf.xacro (robot description, xacro)
@@ -22,4 +22,8 @@
 	    </visual>
     </link>
+ 	<gazebo reference="base_footprint">
+		<material>Gazebo/Blue</material>
+    	<turnGravityOff>false</turnGravityOff>
+  	</gazebo>
 	<joint name="base_footprint_joint" type="fixed">
 		<origin xyz="0 0 0" rpy="0 0 0"/>
@@ -69,4 +73,8 @@
 		</inertial>
 	</link>
+	<gazebo reference="base_link">
+		<material>Gazebo/Blue</material>
+		<turnGravityOff>false</turnGravityOff>
+	</gazebo>
 	<!-- Wheels -->
 	<wheel lr="left" parent="base_link" translateX="0" translateY="${-wheel_y_offset}" translateZ="0" />
@@ -75,4 +83,26 @@
 	<caster fb="front" parent="base_link" translateX="${caster_front_x_offset}" translateY="0" translateZ="${caster_z_offset}" />
 	<caster fb="back" parent="base_link" translateX="${caster_back_x_offset}" translateY="0" translateZ="${caster_z_offset}" />
-	<xacro:include filename="$(find chuck_model)/urdf/chuck.gazebo"/>
+	<!-- Differential drive controller  -->
+	<gazebo>
+		<plugin name="differential_drive_controller" filename="libgazebo_ros_diff_drive.so">
+			<rosDebugLevel>Debug</rosDebugLevel>
+			<publishWheelTF>True</publishWheelTF>
+			<publishTf>1</publishTf>
+			<publishWheelJointState>true</publishWheelJointState>
+			<alwaysOn>true</alwaysOn>
+			<updateRate>100.0</updateRate>
+			<leftJoint>left_wheel_joint</leftJoint>
+			<rightJoint>right_wheel_joint</rightJoint>
+			<wheelSeparation>${2*wheel_y_offset}</wheelSeparation>
+			<wheelDiameter>${2*wheel_radius}</wheelDiameter>
+			<broadcastTF>1</broadcastTF>
+			<wheelTorque>30</wheelTorque>
+			<wheelAcceleration>1.8</wheelAcceleration>
+			<commandTopic>cmd_vel</commandTopic>
+			<odometryFrame>odom</odometryFrame>
+			<odometryTopic>odom</odometryTopic>
+			<robotBaseFrame>base_link</robotBaseFrame>
+		</plugin>
+		<plugin name="gazebo_ros_control" filename="libgazebo_ros_control.so" />
+	</gazebo>
 </robot>

Commit message: Chuck on working map

File: brain/src/chuck_model/urdf/chuck.urdf.xacro (robot description, xacro)
@@ -27,5 +27,5 @@
   	</gazebo>
 	<joint name="base_footprint_joint" type="fixed">
-		<origin xyz="0 0 0" rpy="0 0 0"/>
+		<origin xyz="0 0 ${wheel_radius}" rpy="0 0 0" />
 		<parent link="base_footprint"/>
 		<child link="base_link"/>

Commit message: Fixed chuck model

File: brain/src/chuck_model/urdf/chuck.urdf.xacro (robot description, xacro)
@@ -27,5 +27,5 @@
   	</gazebo>
 	<joint name="base_footprint_joint" type="fixed">
-		<origin xyz="0 0 ${wheel_radius}" rpy="0 0 0" />
+		<origin xyz="0 0 ${base_y_offset + base_z_size/2}" rpy="0 0 0" />
 		<parent link="base_footprint"/>
 		<child link="base_link"/>
@@ -78,6 +78,6 @@
 	</gazebo>
 	<!-- Wheels -->
-	<wheel lr="left" parent="base_link" translateX="0" translateY="${-wheel_y_offset}" translateZ="0" />
-	<wheel lr="right" parent="base_link" translateX="0"  translateY="${wheel_y_offset}" translateZ="0" />
+	<wheel lr="left" parent="base_link" translateX="0" translateY="${-wheel_y_offset}" translateZ="${wheel_z_offset}" />
+	<wheel lr="right" parent="base_link" translateX="0"  translateY="${wheel_y_offset}" translateZ="${wheel_z_offset}" />
 	<!-- Castors -->
 	<caster fb="front" parent="base_link" translateX="${caster_front_x_offset}" translateY="0" translateZ="${caster_z_offset}" />

File: brain/src/chuck_model/urdf/properties.xacro (robot description, xacro)
@@ -9,5 +9,5 @@
 	<xacro:property name="base_y_size" value="0.619125"/>
 	<xacro:property name="base_z_size" value="0.3010916"/>
-	<xacro:property name="base_offset" value="0.070"/>
+	<xacro:property name="base_y_offset" value="0.01905"/>
 	<xacro:property name="base_mass" value="86.1826"/>
 	<!-- Tray support -->
@@ -28,12 +28,12 @@
 	<xacro:property name="tray_zero" value="${support_zero + support_z_size / 2 + tray_z_size / 2}"/>
 	<!-- Wheels -->
-	<xacro:property name="wheel_radius" value="0.2"/>
+	<xacro:property name="wheel_radius" value="0.1016"/>
 	<xacro:property name="wheel_thickness" value="0.047625"/>
 	<xacro:property name="wheel_mass" value="2.118276"/>
 	<xacro:property name="wheel_y_offset" value="0.2661285"/>
-	<xacro:property name="wheel_z_offset" value="0"/>
-	<xacro:property name="caster_radius" value="0.100"/>
-	<xacro:property name="caster_thickness" value="0.025"/>
-	<xacro:property name="caster_mass" value="1.0"/>
+	<xacro:property name="wheel_z_offset" value="${-base_z_size/2 + wheel_radius - base_y_offset}"/>
+	<xacro:property name="caster_radius" value="0.0762"/>
+	<xacro:property name="caster_thickness" value="0.053975"/>
+	<xacro:property name="caster_mass" value="0.453592"/>
 	<xacro:property name="caster_x_size" value="0.1"/>
 	<xacro:property name="caster_y_size" value="0.1"/>
