Commit message: Merge branch 'feature/navigation-motion-controller' into feature/navigation
Conflicts:
	srs_chuck/src/srsbot_chuck/launch/robot.launch
	srs_chuck/src/srsbot_chuck/urdf/sensors/stargazer.urdf.xacro
	srs_chuck/src/srsdrv_stargazer/include/StarGazer.h
	srs_chuck/src/srsdrv_stargazer/src/StarGazer.cpp
	srs_chuck/src/srsdrv_stargazer/src/StarGazerFilter.cpp
	srs_chuck/src/srslib_framework/include/srslib_framework/filter/Sensor.hpp
	srs_chuck/src/srslib_framework/include/srslib_framework/platform/Object.hpp
	srs_chuck/src/srslib_framework/include/srslib_framework/robotics/Odometry.hpp
	srs_chuck/src/srsnode_motion/CMakeLists.txt
	srs_chuck/src/srsnode_motion/include/srsnode_motion/tap/odometry/OdometrySensor.hpp
	srs_chuck/src/srsnode_motion/src/Motion.cpp
	srs_sites/src/srsc_6rhq/map/6rhq-anchors.yaml
	srs_sites/src/srsc_6rhq_norviz/map/6rhq-anchors.yaml
	srs_sites/src/srsc_empty/map/empty-anchors.yaml

File: srs_chuck/src/srsbot_chuck/urdf/sensors/stargazer.urdf.xacro (robot description, xacro)
@@ -6,4 +6,5 @@
   <xacro:property name="stargazer_z_size" value="0.053" />
   <xacro:property name="stargazer_optical_x_offset" value="-0.14" />
+  <xacro:property name="stargazer_optical_y_offset" value="0.0" />
   <xacro:property name="stargazer_optical_y_offset" value="${stargazer_y_size/2}" />
   <xacro:property name="stargazer_optical_z_offset" value="${stargazer_z_size}" />
@@ -23,8 +24,24 @@
       </visual>
     </link>
+    <joint name="stargazer_camera_joint" type="fixed">
+      <parent link="stargazer_link" />
+      <child link="stargazer_camera_frame" />
+      <origin xyz="${stargazer_x_size/2} ${-stargazer_y_size/2} ${stargazer_z_size}" rpy="0 0 0" />
+    </joint>
+	<link name="stargazer_camera_frame">
+  	  <visual>
+       <origin xyz="0 0 0" rpy="0 0 0"/>
+        <geometry>
+         <sphere radius="0.005"/>
+        </geometry>
+        <material name="blue">
+          <color rgba="0 0 1 1"/>
+        </material>
+      </visual>
+    </link>
     <joint name="stargazer_optical_joint" type="fixed">
-      <parent link="stargazer_link" />
+      <parent link="stargazer_camera_frame" />
       <child link="stargazer_optical_frame" />
-      <origin xyz="${stargazer_optical_x_offset + stargazer_x_size/2} ${-stargazer_y_size/2} ${stargazer_z_size}" rpy="0 0 0" />
+      <origin xyz="${stargazer_optical_x_offset} 0 0" rpy="0 0 0" />
     </joint>
 	<link name="stargazer_optical_frame">
