Commit message: Changed to use cleaner logs for shipping

File: srs_chuck/src/srsbot_chuck/urdf/sensors/r200.urdf.xacro (robot description, xacro)
@@ -27,5 +27,5 @@
        <origin xyz="0 0 0" rpy="${M_PI/2} 0 ${M_PI/2}"/>
         <geometry>
-         <mesh filename="package://realsense_navigation/robot_description/meshes/sensors/r200.dae"/>
+          <box size="${r200_cam_x_size} ${r200_cam_y_size} ${r200_cam_z_size}"/>
         </geometry>
       </visual>
