Commit message: Working realsense model integration with live data in rviz

File: srs_chuck/src/srsbot_chuck/urdf/chuck.urdf.xacro (robot description, xacro)
@@ -6,4 +6,5 @@
     <xacro:include filename="component/wheel.urdf.xacro"/>
     <xacro:include filename="component/caster.urdf.xacro"/>
+	<xacro:include filename="sensors/r200.urdf.xacro"/>
     <!-- Robot footprint -->
     <link name="base_footprint">
@@ -83,4 +84,6 @@
     <caster fb="front" parent="base_link" translateX="${caster_front_x_offset}" translateY="0" translateZ="${caster_z_offset}" />
     <caster fb="back" parent="base_link" translateX="${caster_back_x_offset}" translateY="0" translateZ="${caster_z_offset}" />
+	<!-- Realsense R200 -->
+	<sensor_r200 parent="base_link" r200_cam_y_rotation="${M_PI}" r200_cam_px="${base_x_size/2}" r200_cam_py="0" r200_cam_pz="0" />
     <!-- Differential drive controller  -->
     <gazebo>

File: srs_chuck/src/srsbot_chuck/urdf/sensors/r200.urdf.xacro (robot description, xacro)
@@ -7,4 +7,5 @@
   <xacro:property name="r200_cam_rgb_py" value="-0.1034"/>
   <xacro:property name="r200_cam_rgb_pz" value="0.0483"/>
+  <xacro:property name="r200_cam_y_rotation" value="0"/>
   <xacro:property name="r200_cam_depth_offset" value="0.0274"/>
   <!-- Also parameterised in part by the values in turtlebot_properties.urdf.xacro -->
@@ -13,5 +14,5 @@
   parent > camera_rgb_frame
   -->
-  <xacro:macro name="sensor_r200" params="parent r200_cam_px r200_cam_py r200_cam_pz">
+  <xacro:macro name="sensor_r200" params="parent r200_cam_y_rotation r200_cam_px r200_cam_py r200_cam_pz">
     <!--
     ==  RGB joints & links ==
@@ -38,5 +39,5 @@
     <link name="camera_link">
       <visual>
-       <origin xyz="${-r200_cam_rgb_px + -r200_cam_px} ${-r200_cam_rgb_py + -r200_cam_py} ${-r200_cam_rgb_pz + -r200_cam_pz}" rpy="${M_PI/2} 0 ${M_PI/2}"/>
+       <origin xyz="${-r200_cam_rgb_px + -r200_cam_px} ${-r200_cam_rgb_py + -r200_cam_py} ${-r200_cam_rgb_pz + -r200_cam_pz}" rpy="${M_PI/2} ${r200_cam_y_rotation} ${M_PI/2}"/>
         <geometry>
          <mesh filename="package://realsense_navigation/robot_description/meshes/sensors/r200_entire.dae"/>

Commit message: Minor tweaks to filtering

File: srs_chuck/src/srsbot_chuck/urdf/chuck.urdf.xacro (robot description, xacro)
@@ -85,5 +85,5 @@
     <caster fb="back" parent="base_link" translateX="${caster_back_x_offset}" translateY="0" translateZ="${caster_z_offset}" />
 	<!-- Realsense R200 -->
-	<sensor_r200 parent="base_link" r200_cam_y_rotation="${M_PI}" r200_cam_px="${base_x_size/2}" r200_cam_py="0" r200_cam_pz="0" />
+	<sensor_r200 parent="base_link" r200_cam_y_rotation="${M_PI}" r200_cam_px="${base_x_size/2}" r200_cam_py="${-r200_cam_rgb_py/2}" r200_cam_pz="${r200_cam_rgb_pz/2}" />
     <!-- Differential drive controller  -->
     <gazebo>

File: srs_chuck/src/srsbot_chuck/urdf/sensors/r200.urdf.xacro (robot description, xacro)
@@ -41,5 +41,5 @@
        <origin xyz="${-r200_cam_rgb_px + -r200_cam_px} ${-r200_cam_rgb_py + -r200_cam_py} ${-r200_cam_rgb_pz + -r200_cam_pz}" rpy="${M_PI/2} ${r200_cam_y_rotation} ${M_PI/2}"/>
         <geometry>
-         <mesh filename="package://realsense_navigation/robot_description/meshes/sensors/r200_entire.dae"/>
+         <mesh filename="package://realsense_navigation/robot_description/meshes/sensors/r200.dae"/>
         </geometry>
       </visual>

Commit message: Added the concept of trigger to the nodes. It allows synchronous execution of commands on each node. For example, it's now possible for Executive to shut down all the other nodes cleanly.

File: srs_chuck/src/srsbot_chuck/urdf/chuck.urdf.xacro (robot description, xacro)
@@ -1,9 +1,9 @@
 <?xml version="1.0"?>
 <robot name="chuck" xmlns:xacro="http://www.ros.org/wiki/xacro">
-    <xacro:include filename="properties.xacro"/>
-    <xacro:include filename="common/inertia.xacro"/>
-    <xacro:include filename="common/materials.xacro"/>
-    <xacro:include filename="component/wheel.urdf.xacro"/>
-    <xacro:include filename="component/caster.urdf.xacro"/>
+    <xacro:include filename="properties.xacro" />
+    <xacro:include filename="common/inertia.xacro" />
+    <xacro:include filename="common/materials.xacro" />
+    <xacro:include filename="component/wheel.urdf.xacro" />
+    <xacro:include filename="component/caster.urdf.xacro" />
     <!-- Robot footprint -->
     <link name="base_footprint">
@@ -28,47 +28,47 @@
     <joint name="base_footprint_joint" type="fixed">
         <origin xyz="0 0 ${base_y_offset + base_z_size/2}" rpy="0 0 0" />
-        <parent link="base_footprint"/>
-        <child link="base_link"/>
+        <parent link="base_footprint" />
+        <child link="base_link" />
     </joint>
     <!-- Chassis of the robot -->
     <link name="base_link">
         <visual>
-            <origin xyz="0 0 0" rpy="0 0 0"/>
+            <origin xyz="0 0 0" rpy="0 0 0" />
             <geometry>
-                <box size="${base_x_size} ${base_y_size} ${base_z_size}"/>
+                <box size="${base_x_size} ${base_y_size} ${base_z_size}" />
             </geometry>
-            <material name="Blue"/>
+            <material name="Blue" />
         </visual>
         <visual>
-            <origin xyz="0 ${-support_distance / 2} ${support_zero}" rpy="0 0 0"/>
+            <origin xyz="0 ${-support_distance / 2} ${support_zero}" rpy="0 0 0" />
             <geometry>
-                <box size="${support_x_size} ${support_y_size} ${support_z_size}"/>
+                <box size="${support_x_size} ${support_y_size} ${support_z_size}" />
             </geometry>
-            <material name="Blue"/>
+            <material name="Blue" />
         </visual>
         <visual>
-            <origin xyz="0 ${support_distance / 2} ${support_zero}" rpy="0 0 0"/>
+            <origin xyz="0 ${support_distance / 2} ${support_zero}" rpy="0 0 0" />
             <geometry>
-                <box size="${support_x_size} ${support_y_size} ${support_z_size}"/>
+                <box size="${support_x_size} ${support_y_size} ${support_z_size}" />
             </geometry>
-            <material name="Blue"/>
+            <material name="Blue" />
         </visual>
         <visual>
-            <origin xyz="0 0 ${tray_zero}" rpy="0 0 0"/>
+            <origin xyz="0 0 ${tray_zero}" rpy="0 0 0" />
             <geometry>
-                <box size="${tray_x_size} ${tray_y_size} ${tray_z_size}"/>
+                <box size="${tray_x_size} ${tray_y_size} ${tray_z_size}" />
             </geometry>
-            <material name="Blue"/>
+            <material name="Blue" />
         </visual>
         <collision>
-            <origin xyz="0 0 0" rpy="0 0 0"/>
+            <origin xyz="0 0 0" rpy="0 0 0" />
             <geometry>
-                <box size="${base_x_size} ${base_y_size} ${base_z_size}"/>
+                <box size="${base_x_size} ${base_y_size} ${base_z_size}" />
             </geometry>
         </collision>
         <inertial>
-            <mass value="${base_mass}"/>
-            <origin xyz="0 0 0"/>
-            <box_inertia m="${base_mass}" x="${base_x_size}" y="${base_y_size}" z="${base_z_size}"/>
+            <mass value="${base_mass}" />
+            <origin xyz="0 0 0" />
+            <box_inertia m="${base_mass}" x="${base_x_size}" y="${base_y_size}" z="${base_z_size}" />
         </inertial>
     </link>

File: srs_chuck/src/srsbot_chuck/urdf/common/materials.xacro (robot description, xacro)
@@ -2,26 +2,26 @@
 <robot xmlns:xacro="http://www.ros.org/wiki/xacro">
     <material name="Black">
-        <color rgba="0.0 0.0 0.0 1.0"/>
+        <color rgba="0.0 0.0 0.0 1.0" />
     </material>
     <material name="Blue">
-        <color rgba="0.0 0.0 0.8 1.0"/>
+        <color rgba="0.0 0.0 0.8 1.0" />
     </material>
     <material name="Green">
-        <color rgba="0.0 0.8 0.0 1.0"/>
+        <color rgba="0.0 0.8 0.0 1.0" />
     </material>
     <material name="Gray">
-        <color rgba="0.7 0.7 0.7 1.0"/>
+        <color rgba="0.7 0.7 0.7 1.0" />
     </material>
     <material name="DarkGray">
-        <color rgba="0.3 0.3 0.3 1.0"/>
+        <color rgba="0.3 0.3 0.3 1.0" />
     </material>
     <material name="Red">
-        <color rgba="0.8 0.0 0.0 1.0"/>
+        <color rgba="0.8 0.0 0.0 1.0" />
     </material>
     <material name="White">
-        <color rgba="1.0 1.0 1.0 1.0"/>
+        <color rgba="1.0 1.0 1.0 1.0" />
     </material>
     <material name="Yellow">
-        <color rgba="0.8 0.8 0.0 1.0"/>
+        <color rgba="0.8 0.8 0.0 1.0" />
     </material>
 </robot>

File: srs_chuck/src/srsbot_chuck/urdf/component/caster.urdf.xacro (robot description, xacro)
@@ -1,5 +1,5 @@
 <?xml version="1.0"?>
 <robot name="caster" xmlns:xacro="http://www.ros.org/wiki/xacro">
-    <xacro:include filename="common/inertia.xacro"/>
+    <xacro:include filename="common/inertia.xacro" />
     <xacro:macro name="caster" params="fb parent translateX translateY translateZ">
         <link name="${fb}_caster">
@@ -26,7 +26,7 @@
         </link>
         <joint name="caster_${fb}_joint" type="fixed">
-            <parent link="${parent}"/>
-            <child link="${fb}_caster"/>
-            <origin xyz="${translateX} ${translateY} ${translateZ}" rpy="0 0 0"/>
+            <parent link="${parent}" />
+            <child link="${fb}_caster" />
+            <origin xyz="${translateX} ${translateY} ${translateZ}" rpy="0 0 0" />
         </joint>
         <gazebo reference="caster_${fb}_link">

File: srs_chuck/src/srsbot_chuck/urdf/component/wheel.urdf.xacro (robot description, xacro)
@@ -1,5 +1,5 @@
 <?xml version="1.0"?>
 <robot name="wheel" xmlns:xacro="http://www.ros.org/wiki/xacro">
-    <xacro:include filename="common/inertia.xacro"/>
+    <xacro:include filename="common/inertia.xacro" />
     <xacro:macro name="wheel" params="lr parent translateX translateY translateZ">
         <link name="${lr}_wheel">
@@ -7,27 +7,27 @@
                 <origin xyz="0 0 0" rpy="${M_PI/2} 0  0 " />
                 <geometry>
-                    <cylinder length="${wheel_thickness}" radius="${wheel_radius}"/>
+                    <cylinder length="${wheel_thickness}" radius="${wheel_radius}" />
                 </geometry>
-                <material name="Red"/>
+                <material name="Red" />
             </visual>
             <collision>
                 <origin xyz="0 0 0" rpy="${M_PI/2} 0 0 " />
                 <geometry>
-                    <cylinder length="${wheel_thickness}" radius="${wheel_radius}"/>
+                    <cylinder length="${wheel_thickness}" radius="${wheel_radius}" />
                 </geometry>
             </collision>
             <inertial>
-                <mass value="${wheel_mass}"/>
-                <origin xyz="0 0 0"/>
-                <cylinder_inertia m="${wheel_mass}" r="${wheel_radius}" h="${wheel_thickness}"/>
+                <mass value="${wheel_mass}" />
+                <origin xyz="0 0 0" />
+                <cylinder_inertia m="${wheel_mass}" r="${wheel_radius}" h="${wheel_thickness}" />
             </inertial>
         </link>
         <joint name="${lr}_wheel_joint" type="continuous">
-            <parent link="${parent}"/>
-            <child link="${lr}_wheel"/>
-            <origin xyz="${translateX} ${translateY} ${translateZ}" rpy="0 0 0"/>
-            <axis xyz="0 1 0" rpy="0 0 0"/>
-            <limit effort="100" velocity="100"/>
-            <joint_properties damping="0.0" friction="0.0"/>
+            <parent link="${parent}" />
+            <child link="${lr}_wheel" />
+            <origin xyz="${translateX} ${translateY} ${translateZ}" rpy="0 0 0" />
+            <axis xyz="0 1 0" rpy="0 0 0" />
+            <limit effort="100" velocity="100" />
+            <joint_properties damping="0.0" friction="0.0" />
         </joint>
         <transmission name="${lr}_wheel_joint_trans">
@@ -42,9 +42,9 @@
         </transmission>
         <gazebo reference="${lr}_wheel">
-            <mu1 value="1.0"/>
-            <mu2 value="1.0"/>
-            <kp  value="10000000.0"/>
-            <kd  value="1.0"/>
-            <fdir1 value="1 0 0"/>
+            <mu1 value="1.0" />
+            <mu2 value="1.0" />
+            <kp  value="10000000.0" />
+            <kd  value="1.0" />
+            <fdir1 value="1 0 0" />
             <material>Gazebo/White</material>
             <turnGravityOff>false</turnGravityOff>

File: srs_chuck/src/srsbot_chuck/urdf/properties.xacro (robot description, xacro)
@@ -2,43 +2,43 @@
 <robot name="chuck" xmlns:xacro="http://www.ros.org/wiki/xacro">
     <!-- All units in m-kg-s-radians unit system -->
-    <xacro:property name="M_PI" value="3.1415926535897931"/>
+    <xacro:property name="M_PI" value="3.1415926535897931" />
     <xacro:property name="M_PI_2" value="1.570796327" />
     <xacro:property name="DEG_TO_RAD" value="0.017453293" />
     <!-- Chassis -->
-    <xacro:property name="base_x_size" value="0.9772396"/>
-    <xacro:property name="base_y_size" value="0.619125"/>
-    <xacro:property name="base_z_size" value="0.3010916"/>
-    <xacro:property name="base_y_offset" value="0.01905"/>
-    <xacro:property name="base_mass" value="86.1826"/>
+    <xacro:property name="base_x_size" value="0.9772396" />
+    <xacro:property name="base_y_size" value="0.619125" />
+    <xacro:property name="base_z_size" value="0.3010916" />
+    <xacro:property name="base_y_offset" value="0.01905" />
+    <xacro:property name="base_mass" value="86.1826" />
     <!-- Tray support -->
-    <xacro:property name="support_x_size" value="0.050"/>
-    <xacro:property name="support_y_size" value="0.050"/>
-    <xacro:property name="support_z_size" value="0.600"/>
-    <xacro:property name="support_distance" value="0.254"/>
-    <xacro:property name="tray_x_size" value="0.863"/>
-    <xacro:property name="tray_y_size" value="0.635"/>
-    <xacro:property name="tray_z_size" value="0.038"/>
-    <xacro:property name="screen_x_size" value="0.020"/>
-    <xacro:property name="screen_y_size" value="0.300"/>
-    <xacro:property name="screen_z_size" value="0.200"/>
-    <xacro:property name="screen_inclination" value="0.200"/>
-    <xacro:property name="screen_mass" value="0.500"/>
-    <xacro:property name="body_zero" value="0"/>
-    <xacro:property name="support_zero" value="${body_zero + base_z_size / 2 + support_z_size / 2}"/>
-    <xacro:property name="tray_zero" value="${support_zero + support_z_size / 2 + tray_z_size / 2}"/>
+    <xacro:property name="support_x_size" value="0.050" />
+    <xacro:property name="support_y_size" value="0.050" />
+    <xacro:property name="support_z_size" value="0.600" />
+    <xacro:property name="support_distance" value="0.254" />
+    <xacro:property name="tray_x_size" value="0.863" />
+    <xacro:property name="tray_y_size" value="0.635" />
+    <xacro:property name="tray_z_size" value="0.038" />
+    <xacro:property name="screen_x_size" value="0.020" />
+    <xacro:property name="screen_y_size" value="0.300" />
+    <xacro:property name="screen_z_size" value="0.200" />
+    <xacro:property name="screen_inclination" value="0.200" />
+    <xacro:property name="screen_mass" value="0.500" />
+    <xacro:property name="body_zero" value="0" />
+    <xacro:property name="support_zero" value="${body_zero + base_z_size / 2 + support_z_size / 2}" />
+    <xacro:property name="tray_zero" value="${support_zero + support_z_size / 2 + tray_z_size / 2}" />
     <!-- Wheels -->
-    <xacro:property name="wheel_radius" value="0.1016"/>
-    <xacro:property name="wheel_thickness" value="0.047625"/>
-    <xacro:property name="wheel_mass" value="2.118276"/>
-    <xacro:property name="wheel_y_offset" value="0.2661285"/>
-    <xacro:property name="wheel_z_offset" value="${-base_z_size/2 + wheel_radius - base_y_offset}"/>
-    <xacro:property name="caster_radius" value="0.0762"/>
-    <xacro:property name="caster_thickness" value="0.053975"/>
-    <xacro:property name="caster_mass" value="0.453592"/>
-    <xacro:property name="caster_x_size" value="0.1"/>
-    <xacro:property name="caster_y_size" value="0.1"/>
-    <xacro:property name="caster_z_size" value="0.2"/>
-    <xacro:property name="caster_front_x_offset" value="0.2885948"/>
-    <xacro:property name="caster_back_x_offset" value="-0.3564382"/>
-    <xacro:property name="caster_z_offset" value="${wheel_z_offset - (wheel_radius - caster_radius) + 0.0001 }"/>
+    <xacro:property name="wheel_radius" value="0.1016" />
+    <xacro:property name="wheel_thickness" value="0.047625" />
+    <xacro:property name="wheel_mass" value="2.118276" />
+    <xacro:property name="wheel_y_offset" value="0.2661285" />
+    <xacro:property name="wheel_z_offset" value="${-base_z_size/2 + wheel_radius - base_y_offset}" />
+    <xacro:property name="caster_radius" value="0.0762" />
+    <xacro:property name="caster_thickness" value="0.053975" />
+    <xacro:property name="caster_mass" value="0.453592" />
+    <xacro:property name="caster_x_size" value="0.1" />
+    <xacro:property name="caster_y_size" value="0.1" />
+    <xacro:property name="caster_z_size" value="0.2" />
+    <xacro:property name="caster_front_x_offset" value="0.2885948" />
+    <xacro:property name="caster_back_x_offset" value="-0.3564382" />
+    <xacro:property name="caster_z_offset" value="${wheel_z_offset - (wheel_radius - caster_radius) + 0.0001 }" />
 </robot>

File: srs_chuck/src/srsbot_chuck/urdf/sensors/r200.urdf.xacro (robot description, xacro)
@@ -1,11 +1,11 @@
 <?xml version="1.0"?>
 <robot name="sensor_r200" xmlns:xacro="http://ros.org/wiki/xacro">
-  <xacro:include filename="$(find turtlebot_description)/urdf/turtlebot_gazebo.urdf.xacro"/>
-  <xacro:include filename="$(find turtlebot_description)/urdf/turtlebot_properties.urdf.xacro"/>
+  <xacro:include filename="$(find turtlebot_description)/urdf/turtlebot_gazebo.urdf.xacro" />
+  <xacro:include filename="$(find turtlebot_description)/urdf/turtlebot_properties.urdf.xacro" />
   <!-- Following values measured on the 3d model -->
-  <xacro:property name="r200_cam_rgb_px" value="0.0088"/>
-  <xacro:property name="r200_cam_rgb_py" value="-0.1034"/>
-  <xacro:property name="r200_cam_rgb_pz" value="0.0483"/>
-  <xacro:property name="r200_cam_depth_offset" value="0.0274"/>
+  <xacro:property name="r200_cam_rgb_px" value="0.0088" />
+  <xacro:property name="r200_cam_rgb_py" value="-0.1034" />
+  <xacro:property name="r200_cam_rgb_pz" value="0.0483" />
+  <xacro:property name="r200_cam_depth_offset" value="0.0274" />
   <!-- Also parameterised in part by the values in turtlebot_properties.urdf.xacro -->
   <!--
@@ -18,9 +18,9 @@
     -->
     <joint name="camera_rgb_joint" type="fixed">
-      <origin xyz="${r200_cam_rgb_px + r200_cam_px} ${r200_cam_rgb_py + r200_cam_py} ${r200_cam_rgb_pz + r200_cam_pz}" rpy="0 0 0"/>
-      <parent link="${parent}"/>
+      <origin xyz="${r200_cam_rgb_px + r200_cam_px} ${r200_cam_rgb_py + r200_cam_py} ${r200_cam_rgb_pz + r200_cam_pz}" rpy="0 0 0" />
+      <parent link="${parent}" />
       <child link="camera_rgb_frame" />
     </joint>
-    <link name="camera_rgb_frame"/>
+    <link name="camera_rgb_frame" />
     <joint name="camera_rgb_optical_joint" type="fixed">
       <origin xyz="0 0 0" rpy="${-M_PI/2} 0 ${-M_PI/2}" />
@@ -28,23 +28,23 @@
       <child link="camera_rgb_optical_frame" />
     </joint>
-    <link name="camera_rgb_optical_frame"/>
+    <link name="camera_rgb_optical_frame" />
     <!-- Placing the camera joint -->
     <joint name="camera_joint" type="fixed">
-      <origin xyz="${r200_cam_px} ${r200_cam_py} ${r200_cam_pz}" rpy="${cam_or} ${cam_op} ${cam_oy}"/>
-      <parent link="camera_rgb_frame"/>
-      <child link="camera_link"/>
+      <origin xyz="${r200_cam_px} ${r200_cam_py} ${r200_cam_pz}" rpy="${cam_or} ${cam_op} ${cam_oy}" />
+      <parent link="camera_rgb_frame" />
+      <child link="camera_link" />
     </joint>
     <!-- Mounting the camera at the right position -->
     <link name="camera_link">
       <visual>
-       <origin xyz="${-r200_cam_rgb_px + -r200_cam_px} ${-r200_cam_rgb_py + -r200_cam_py} ${-r200_cam_rgb_pz + -r200_cam_pz}" rpy="${M_PI/2} 0 ${M_PI/2}"/>
+       <origin xyz="${-r200_cam_rgb_px + -r200_cam_px} ${-r200_cam_rgb_py + -r200_cam_py} ${-r200_cam_rgb_pz + -r200_cam_pz}" rpy="${M_PI/2} 0 ${M_PI/2}" />
         <geometry>
-         <mesh filename="package://realsense_navigation/robot_description/meshes/sensors/r200_entire.dae"/>
+         <mesh filename="package://realsense_navigation/robot_description/meshes/sensors/r200_entire.dae" />
         </geometry>
       </visual>
       <collision>
-        <origin xyz="0.0 0.0 0.0" rpy="0 0 0"/>
+        <origin xyz="0.0 0.0 0.0" rpy="0 0 0" />
         <geometry>
-          <box size="0.130 0.567 0.118"/>
+          <box size="0.130 0.567 0.118" />
         </geometry>
       </collision>
@@ -66,5 +66,5 @@
   	  <child link="camera_depth_frame" />
   	</joint>
-  	<link name="camera_depth_frame"/>
+  	<link name="camera_depth_frame" />
   	<joint name="camera_depth_optical_joint" type="fixed">
   	  <origin xyz="0 0 0" rpy="${-M_PI/2} 0 ${-M_PI/2}" />
@@ -72,5 +72,5 @@
   	  <child link="camera_depth_optical_frame" />
   	</joint>
-  	<link name="camera_depth_optical_frame"/>
+  	<link name="camera_depth_optical_frame" />
   	<turtlebot_sim_3dsensor/>
   </xacro:macro>
