Commit message: Fixed realsense model

File: srs_chuck/src/srsbot_chuck/urdf/chuck.urdf.xacro (robot description, xacro)
@@ -28,5 +28,5 @@
       </gazebo>
     <joint name="base_footprint_joint" type="fixed">
-        <origin xyz="0 0 ${base_y_offset + base_z_size/2}" rpy="0 0 0" />
+        <origin xyz="0 0 ${base_z_offset + base_z_size/2}" rpy="0 0 0" />
         <parent link="base_footprint" />
         <child link="base_link" />
@@ -85,5 +85,5 @@
     <caster fb="back" parent="base_link" translateX="${caster_back_x_offset}" translateY="0" translateZ="${caster_z_offset}" />
 	<!-- Realsense R200 -->
-	<sensor_r200 parent="base_link" r200_cam_y_rotation="${M_PI}" r200_cam_px="${base_x_size/2}" r200_cam_py="${-r200_cam_rgb_py/2}" r200_cam_pz="${r200_cam_rgb_pz/2}" />
+	<sensor_r200 parent="base_link" r200_cam_y_rotation="${M_PI}" r200_cam_px="${base_x_size/2}" r200_cam_py="${r200_cam_y_size/2}" r200_cam_pz="${r200_cam_z_size + realsense_z_offset}" />
     <!-- Differential drive controller  -->
     <gazebo>

File: srs_chuck/src/srsbot_chuck/urdf/properties.xacro (robot description, xacro)
@@ -9,5 +9,5 @@
     <xacro:property name="base_y_size" value="0.619125" />
     <xacro:property name="base_z_size" value="0.3010916" />
-    <xacro:property name="base_y_offset" value="0.01905" />
+    <xacro:property name="base_z_offset" value="0.01905" />
     <xacro:property name="base_mass" value="86.1826" />
     <!-- Tray support -->
@@ -32,5 +32,5 @@
     <xacro:property name="wheel_mass" value="2.118276" />
     <xacro:property name="wheel_y_offset" value="0.2661285" />
-    <xacro:property name="wheel_z_offset" value="${-base_z_size/2 + wheel_radius - base_y_offset}" />
+    <xacro:property name="wheel_z_offset" value="${-base_z_size/2 + wheel_radius - base_z_offset}" />
     <xacro:property name="caster_radius" value="0.0762" />
     <xacro:property name="caster_thickness" value="0.053975" />
@@ -42,3 +42,5 @@
     <xacro:property name="caster_back_x_offset" value="-0.3564382" />
     <xacro:property name="caster_z_offset" value="${wheel_z_offset - (wheel_radius - caster_radius) + 0.0001 }" />
+    <!-- Sensors -->
+	<xacro:property name="realsense_z_offset" value="0.0641858" />
 </robot>

File: srs_chuck/src/srsbot_chuck/urdf/sensors/r200.urdf.xacro (robot description, xacro)
@@ -4,9 +4,12 @@
   <xacro:include filename="$(find turtlebot_description)/urdf/turtlebot_properties.urdf.xacro" />
   <!-- Following values measured on the 3d model -->
-  <xacro:property name="r200_cam_rgb_px" value="0.0088" />
-  <xacro:property name="r200_cam_rgb_py" value="-0.1034" />
-  <xacro:property name="r200_cam_rgb_pz" value="0.0483" />
-  <xacro:property name="r200_cam_y_rotation" value="0" />
-  <xacro:property name="r200_cam_depth_offset" value="0.0274" />
+  <xacro:property name="r200_cam_x_size" value="0.00759" />
+  <xacro:property name="r200_cam_y_size" value="0.130" />
+  <xacro:property name="r200_cam_z_size" value="0.01936" />
+  <!-- Following values measured on the 3d model -->
+  <xacro:property name="r200_cam_rgb_x_offset" value="0.00425"/>
+  <xacro:property name="r200_cam_rgb_y_offset" value="0.01954"/>
+  <xacro:property name="r200_cam_rgb_z_offset" value="0.01334"/>
+  <xacro:property name="r200_cam_depth_offset" value="0.0274"/>
   <!-- Also parameterised in part by the values in turtlebot_properties.urdf.xacro -->
   <!--
@@ -14,30 +17,15 @@
   parent > camera_rgb_frame
   -->
-  <xacro:macro name="sensor_r200" params="parent r200_cam_y_rotation r200_cam_px r200_cam_py r200_cam_pz">
-    <!--
-    ==  RGB joints & links ==
-    -->
-    <joint name="camera_rgb_joint" type="fixed">
-      <origin xyz="${r200_cam_rgb_px + r200_cam_px} ${r200_cam_rgb_py + r200_cam_py} ${r200_cam_rgb_pz + r200_cam_pz}" rpy="0 0 0" />
-      <parent link="${parent}" />
-      <child link="camera_rgb_frame" />
-    </joint>
-    <link name="camera_rgb_frame" />
-    <joint name="camera_rgb_optical_joint" type="fixed">
-      <origin xyz="0 0 0" rpy="${-M_PI/2} 0 ${-M_PI/2}" />
-      <parent link="camera_rgb_frame" />
-      <child link="camera_rgb_optical_frame" />
-    </joint>
-    <link name="camera_rgb_optical_frame" />
+  <xacro:macro name="sensor_r200" params="parent r200_cam_px r200_cam_py r200_cam_pz r200_cam_y_rotation">
     <!-- Placing the camera joint -->
     <joint name="camera_joint" type="fixed">
-      <origin xyz="${r200_cam_px} ${r200_cam_py} ${r200_cam_pz}" rpy="${cam_or} ${cam_op} ${cam_oy}" />
-      <parent link="camera_rgb_frame" />
-      <child link="camera_link" />
+      <origin xyz="${r200_cam_px} ${r200_cam_py} ${r200_cam_pz}" rpy="${r200_cam_y_rotation} 0 0"/>
+      <parent link="${parent}"/>
+      <child link="camera_link"/>
     </joint>
     <!-- Mounting the camera at the right position -->
     <link name="camera_link">
       <visual>
-       <origin xyz="${-r200_cam_rgb_px + -r200_cam_px} ${-r200_cam_rgb_py + -r200_cam_py} ${-r200_cam_rgb_pz + -r200_cam_pz}" rpy="${M_PI/2} ${r200_cam_y_rotation} ${M_PI/2}"/>
+       <origin xyz="0 0 0" rpy="${M_PI/2} 0 ${M_PI/2}"/>
         <geometry>
          <mesh filename="package://realsense_navigation/robot_description/meshes/sensors/r200.dae"/>
@@ -45,7 +33,7 @@
       </visual>
       <collision>
-        <origin xyz="0.0 0.0 0.0" rpy="0 0 0" />
+        <origin xyz="${r200_cam_x_size/2} ${r200_cam_y_size/2} ${r200_cam_z_size/2}" rpy="0 0 0"/>
         <geometry>
-          <box size="0.130 0.567 0.118" />
+          <box size="${r200_cam_x_size} ${r200_cam_y_size} ${r200_cam_z_size}"/>
         </geometry>
       </collision>
@@ -60,12 +48,47 @@
     </link>
     <!--
+    ==  RGB joints & links ==
+    -->
+    <joint name="camera_rgb_joint" type="fixed">
+      <origin xyz="${r200_cam_rgb_x_offset} ${r200_cam_rgb_y_offset} ${r200_cam_rgb_z_offset}" rpy="0 0 0"/>
+      <parent link="camera_link"/>
+      <child link="camera_rgb_frame" />
+    </joint>
+    <link name="camera_rgb_frame">
+      <visual>
+       <origin xyz="0 0 0" rpy="${M_PI/2} 0 ${M_PI/2}"/>
+        <geometry>
+         <sphere radius="0.005"/>
+        </geometry>
+        <material name="green">
+          <color rgba="0 1 0 1"/>
+        </material>
+      </visual>
+    </link>
+    <joint name="camera_rgb_optical_joint" type="fixed">
+      <origin xyz="0 0 0" rpy="${-M_PI/2} 0 ${-M_PI/2}" />
+      <parent link="camera_rgb_frame" />
+      <child link="camera_rgb_optical_frame" />
+    </joint>
+    <link name="camera_rgb_optical_frame"/>
+    <!--
     ==  Depth joints & links ==
     -->
   	<joint name="camera_depth_joint" type="fixed">
-  	  <origin xyz="0 ${r200_cam_depth_offset} 0" rpy="0 0 0" />
-  	  <parent link="camera_rgb_frame" />
+  	  <origin xyz="${r200_cam_rgb_x_offset} ${r200_cam_rgb_y_offset+r200_cam_depth_offset} ${r200_cam_rgb_z_offset}" rpy="0 0 0" />
+  	  <parent link="camera_link" />
   	  <child link="camera_depth_frame" />
   	</joint>
-  	<link name="camera_depth_frame" />
+  	<link name="camera_depth_frame">
+  	  <visual>
+       <origin xyz="0 0 0" rpy="${M_PI/2} 0 ${M_PI/2}"/>
+        <geometry>
+         <sphere radius="0.005"/>
+        </geometry>
+        <material name="green">
+          <color rgba="0 0 1 1"/>
+        </material>
+      </visual>
+  	</link>
   	<joint name="camera_depth_optical_joint" type="fixed">
   	  <origin xyz="0 0 0" rpy="${-M_PI/2} 0 ${-M_PI/2}" />
@@ -73,5 +96,5 @@
   	  <child link="camera_depth_optical_frame" />
   	</joint>
-  	<link name="camera_depth_optical_frame" />
+  	<link name="camera_depth_optical_frame"/>
   	<turtlebot_sim_3dsensor/>
   </xacro:macro>

Commit message: Stargazer transform fixes. Added back in circleci file. Implemented some of the new brainstem messages.

File: srs_chuck/src/srsbot_chuck/urdf/chuck.urdf.xacro (robot description, xacro)
@@ -7,4 +7,5 @@
     <xacro:include filename="component/caster.urdf.xacro" />
 	<xacro:include filename="sensors/r200.urdf.xacro"/>
+	<xacro:include filename="sensors/stargazer.urdf.xacro"/>
     <!-- Robot footprint -->
     <link name="base_footprint">
@@ -28,5 +29,5 @@
       </gazebo>
     <joint name="base_footprint_joint" type="fixed">
-        <origin xyz="0 0 ${base_z_offset + base_z_size/2}" rpy="0 0 0" />
+        <origin xyz="0 0 ${base_footprint_z_offset}" rpy="0 0 0" />
         <parent link="base_footprint" />
         <child link="base_link" />
@@ -85,5 +86,23 @@
     <caster fb="back" parent="base_link" translateX="${caster_back_x_offset}" translateY="0" translateZ="${caster_z_offset}" />
 	<!-- Realsense R200 -->
-	<sensor_r200 parent="base_link" r200_cam_y_rotation="${M_PI}" r200_cam_px="${base_x_size/2}" r200_cam_py="${r200_cam_y_size/2}" r200_cam_pz="${r200_cam_z_size + realsense_z_offset}" />
+	<sensor_r200 parent="base_link" r200_cam_y_rotation="${M_PI}" r200_cam_px="${r200_x_offset}" r200_cam_py="${r200_y_offset}" r200_cam_pz="${r200_z_offset}" />
+	<!-- Stargazer -->
+	<stargazer parent="base_link" translateX="${stargazer_x_offset}" translateY="${stargazer_y_offset}" translateZ="${stargazer_z_offset}" />
+  	<joint name="laser_frame_joint" type="fixed">
+  	  <origin xyz="${base_x_size/2} 0 0" rpy="0 0 0" />
+  	  <parent link="base_footprint" />
+  	  <child link="laser_frame" />
+  	</joint>
+  	<link name="laser_frame" >
+      <visual>
+       <origin xyz="0 0 0" rpy="0 0 0"/>
+        <geometry>
+         <sphere radius="0.005"/>
+        </geometry>
+        <material name="orange">
+          <color rgba="0 0 1 1"/>
+        </material>
+      </visual>
+  	</link>
     <!-- Differential drive controller  -->
     <gazebo>

File: srs_chuck/src/srsbot_chuck/urdf/properties.xacro (robot description, xacro)
@@ -11,4 +11,5 @@
     <xacro:property name="base_z_offset" value="0.01905" />
     <xacro:property name="base_mass" value="86.1826" />
+	<xacro:property name="base_footprint_z_offset" value="${base_z_offset + base_z_size/2}" />
     <!-- Tray support -->
     <xacro:property name="support_x_size" value="0.050" />
@@ -42,5 +43,15 @@
     <xacro:property name="caster_back_x_offset" value="-0.3564382" />
     <xacro:property name="caster_z_offset" value="${wheel_z_offset - (wheel_radius - caster_radius) + 0.0001 }" />
+    <!-- Realsense Position (relative to base_link) -->
+    <xacro:property name="r200_x_offset" value="${base_x_size/2}" />
+    <xacro:property name="r200_y_offset" value="${r200_cam_y_size/2}" />
+    <xacro:property name="r200_z_offset" value="${r200_cam_z_size + realsense_z_offset}" />
     <!-- Sensors -->
+    <!-- Realsense -->
 	<xacro:property name="realsense_z_offset" value="0.0641858" />
+    <!-- Stargazer -->
+    <!-- All measurements made from base_link -> bottom left corner of stargazer -->
+	<xacro:property name="stargazer_x_offset" value="-0.4217162" />
+	<xacro:property name="stargazer_y_offset" value="-0.0352552" />
+	<xacro:property name="stargazer_z_offset" value="0.998982" />
 </robot>

Commit message: Fixed bug in urdf

File: srs_chuck/src/srsbot_chuck/urdf/chuck.urdf.xacro (robot description, xacro)
@@ -10,11 +10,4 @@
     <!-- Robot footprint -->
     <link name="base_footprint">
-        <inertial>
-          <mass value="0.0001" />
-          <origin xyz="0 0 0" />
-          <inertia ixx="0.0001" ixy="0.0" ixz="0.0"
-              iyy="0.0001" iyz="0.0"
-              izz="0.0001" />
-        </inertial>
         <visual>
             <origin xyz="0 0 0" rpy="0 0 0" />

Commit message: Fixed robot model

File: srs_chuck/src/srsbot_chuck/urdf/chuck.urdf.xacro (robot description, xacro)
@@ -99,5 +99,10 @@
       </visual>
   	</link>
-  	<xacro:sick_tim310 name="laser" ros_topic="scan" />
+    <sick_tim551 name="sick_lidar" ros_topic="scan" />
+  	<joint name="lidar_laser_frame_joint" type="fixed">
+  	  <origin xyz="${base_x_size/2} 0 0" rpy="0 0 0" />
+  	  <parent link="base_footprint" />
+  	  <child link="sick_lidar_mount_link" />
+  	</joint>
     <!-- Differential drive controller  -->
     <gazebo>

Commit message: Flipped lidar right side up

File: srs_chuck/src/srsbot_chuck/urdf/chuck.urdf.xacro (robot description, xacro)
@@ -101,5 +101,5 @@
     <sick_tim551 name="sick_lidar" ros_topic="scan" />
   	<joint name="lidar_laser_frame_joint" type="fixed">
-  	  <origin xyz="${base_x_size/2} 0 0" rpy="0 0 0" />
+  	  <origin xyz="${base_x_size/2} 0 0" rpy="${M_PI} 0 0" />
   	  <parent link="base_footprint" />
   	  <child link="sick_lidar_mount_link" />

Commit message: Added corrected lidar offsets

File: srs_chuck/src/srsbot_chuck/urdf/chuck.urdf.xacro (robot description, xacro)
@@ -101,5 +101,5 @@
     <sick_tim551 name="sick_lidar" ros_topic="scan" />
   	<joint name="lidar_laser_frame_joint" type="fixed">
-  	  <origin xyz="${base_x_size/2} 0 0" rpy="${M_PI} 0 0" />
+      <origin xyz="${lidar_x_offset} 0 0" rpy="${M_PI} 0 0" />
   	  <parent link="base_footprint" />
   	  <child link="sick_lidar_mount_link" />

File: srs_chuck/src/srsbot_chuck/urdf/properties.xacro (robot description, xacro)
@@ -55,3 +55,5 @@
 	<xacro:property name="stargazer_y_offset" value="-0.0352552" />
 	<xacro:property name="stargazer_z_offset" value="0.998982" />
+	<!-- SICK Lidar -->
+	<xacro:property name="lidar_x_offset" value="0.4600448" />
 </robot>

Commit message: Added new calibration for pollux and boris.

File: srs_chuck/src/srsbot_chuck/urdf/chuck.urdf.xacro (robot description, xacro)
@@ -8,4 +8,5 @@
 	<xacro:include filename="sensors/r200.urdf.xacro"/>
 	<xacro:include filename="sensors/stargazer.urdf.xacro"/>
+	<xacro:include filename="$(find sick_tim)/urdf/sick_tim.urdf.xacro" />
     <!-- Robot footprint -->
     <link name="base_footprint">
@@ -98,4 +99,10 @@
       </visual>
   	</link>
+    <sick_tim551 name="sick_lidar" ros_topic="scan" />
+  	<joint name="lidar_laser_frame_joint" type="fixed">
+      <origin xyz="${lidar_x_offset} 0 0" rpy="${M_PI} 0 0" />
+  	  <parent link="base_footprint" />
+  	  <child link="sick_lidar_mount_link" />
+  	</joint>
     <!-- Differential drive controller  -->
     <gazebo>

Commit message: Removed sick lidar from robot model and launch file (until chuck 2.0 is released).

File: srs_chuck/src/srsbot_chuck/urdf/chuck.urdf.xacro (robot description, xacro)
@@ -8,5 +8,5 @@
 	<xacro:include filename="sensors/r200.urdf.xacro"/>
 	<xacro:include filename="sensors/stargazer.urdf.xacro"/>
-	<xacro:include filename="$(find sick_tim)/urdf/sick_tim.urdf.xacro" />
+	<!-- <xacro:include filename="$(find sick_tim)/urdf/sick_tim.urdf.xacro" /> -->
     <!-- Robot footprint -->
     <link name="base_footprint">
@@ -99,10 +99,10 @@
       </visual>
   	</link>
-    <sick_tim551 name="sick_lidar" ros_topic="scan" />
+    <!-- <sick_tim551 name="sick_lidar" ros_topic="scan" />
   	<joint name="lidar_laser_frame_joint" type="fixed">
       <origin xyz="${lidar_x_offset} 0 0" rpy="${M_PI} 0 0" />
   	  <parent link="base_footprint" />
   	  <child link="sick_lidar_mount_link" />
-  	</joint>
+  	</joint> -->
     <!-- Differential drive controller  -->
     <gazebo>

Commit message: Backed out changes to imu branch (should have been sep branch).

File: srs_chuck/src/srsbot_chuck/urdf/chuck.urdf.xacro (robot description, xacro)
@@ -8,5 +8,4 @@
 	<xacro:include filename="sensors/r200.urdf.xacro"/>
 	<xacro:include filename="sensors/stargazer.urdf.xacro"/>
-	<!-- <xacro:include filename="$(find sick_tim)/urdf/sick_tim.urdf.xacro" /> -->
     <!-- Robot footprint -->
     <link name="base_footprint">
@@ -99,10 +98,4 @@
       </visual>
   	</link>
-    <!-- <sick_tim551 name="sick_lidar" ros_topic="scan" />
-  	<joint name="lidar_laser_frame_joint" type="fixed">
-      <origin xyz="${lidar_x_offset} 0 0" rpy="${M_PI} 0 0" />
-  	  <parent link="base_footprint" />
-  	  <child link="sick_lidar_mount_link" />
-  	</joint> -->
     <!-- Differential drive controller  -->
     <gazebo>

File: srs_chuck/src/srsbot_chuck/urdf/properties.xacro (robot description, xacro)
@@ -55,5 +55,3 @@
 	<xacro:property name="stargazer_y_offset" value="-0.0352552" />
 	<xacro:property name="stargazer_z_offset" value="0.998982" />
-	<!-- SICK Lidar -->
-	<xacro:property name="lidar_x_offset" value="0.4600448" />
 </robot>

Commit message: More nav/localiation fixes

File: srs_chuck/src/srsbot_chuck/urdf/chuck.urdf.xacro (robot description, xacro)
@@ -101,5 +101,5 @@
     <sick_tim551 name="sick_lidar" ros_topic="scan" />
   	<joint name="lidar_laser_frame_joint" type="fixed">
-      <origin xyz="${lidar_x_offset} 0 0" rpy="${M_PI} 0 0" />
+      <origin xyz="${lidar_x_offset} 0 ${lidar_z_offset}" rpy="${M_PI} 0 0" />
   	  <parent link="base_footprint" />
   	  <child link="sick_lidar_mount_link" />

File: srs_chuck/src/srsbot_chuck/urdf/properties.xacro (robot description, xacro)
@@ -57,3 +57,4 @@
 	<!-- SICK Lidar -->
 	<xacro:property name="lidar_x_offset" value="0.4600448" />
+	<xacro:property name="lidar_z_offset" value="0.3175" />
 </robot>

Commit message: Major overhaul of navigation stack tuning in challenging environment

File: srs_chuck/src/srsbot_chuck/urdf/chuck.urdf.xacro (robot description, xacro)
@@ -1,5 +1,5 @@
 <?xml version="1.0"?>
 <robot name="chuck" xmlns:xacro="http://www.ros.org/wiki/xacro">
-    <xacro:include filename="properties.xacro" />
+    <xacro:include filename="$(env HOME)/mfp_robot_config/robot_properties.xacro" />
     <xacro:include filename="common/inertia.xacro" />
     <xacro:include filename="common/materials.xacro" />
@@ -101,5 +101,5 @@
     <sick_tim551 name="sick_lidar" ros_topic="scan" />
   	<joint name="lidar_laser_frame_joint" type="fixed">
-      <origin xyz="${lidar_x_offset} 0 ${lidar_z_offset}" rpy="${M_PI} 0 0" />
+      <origin xyz="${lidar_x_offset} 0 ${lidar_z_offset}" rpy="${lidar_rotation} 0 0" />
   	  <parent link="base_footprint" />
   	  <child link="sick_lidar_mount_link" />

Commit message: change chuck urdf to flip laser_frame because we actually setup realsense upside down

File: srs_chuck/src/srsbot_chuck/urdf/chuck.urdf.xacro (robot description, xacro)
@@ -84,5 +84,5 @@
 	<stargazer parent="base_link" translateX="${stargazer_x_offset}" translateY="${stargazer_y_offset}" translateZ="${stargazer_z_offset}" />
   	<joint name="laser_frame_joint" type="fixed">
-  	  <origin xyz="${base_x_size/2} 0 0" rpy="0 0 0" />
+  	  <origin xyz="${base_x_size/2} 0 0" rpy="${M_PI} 0 0" />
   	  <parent link="base_footprint" />
   	  <child link="laser_frame" />

Commit message: Fix urdf for speckles

File: srs_chuck/src/srsbot_chuck/urdf/chuck.urdf.xacro (robot description, xacro)
@@ -80,9 +80,7 @@
     <caster fb="back" parent="base_link" translateX="${caster_back_x_offset}" translateY="0" translateZ="${caster_z_offset}" />
 	<!-- Realsense R200 -->
-	<sensor_r200 parent="base_link" r200_cam_y_rotation="${M_PI}" r200_cam_px="${r200_x_offset}" r200_cam_py="${r200_y_offset}" r200_cam_pz="${r200_z_offset}" />
-	<!-- Stargazer -->
-	<stargazer parent="base_link" translateX="${stargazer_x_offset}" translateY="${stargazer_y_offset}" translateZ="${stargazer_z_offset}" />
+	<sensor_r200 parent="base_link" r200_cam_y_rotation="${realsense_z_rotation}" r200_cam_px="${r200_x_offset}" r200_cam_py="${r200_y_offset}" r200_cam_pz="${r200_z_offset}" />
   	<joint name="laser_frame_joint" type="fixed">
-  	  <origin xyz="${base_x_size/2} 0 0" rpy="${M_PI} 0 0" />
+  	  <origin xyz="${base_x_size/2} 0 0" rpy="${realsense_z_rotation} 0 0" />
   	  <parent link="base_footprint" />
   	  <child link="laser_frame" />
