Commit message: modify realsense urdf and resolve conflict

File: srs_chuck/src/srsbot_chuck/urdf/config/robot_properties.xacro (robot description, xacro)
@@ -49,5 +49,5 @@
     <!-- Sensors -->
     <!-- Realsense -->
-    <xacro:property name="realsense_z_offset" value="0.0641858" />
+    <xacro:property name="realsense_z_offset" value="-0.09766" />
     <!-- Stargazer -->
     <!-- All measurements made from base_link -> bottom left corner of stargazer -->

Commit message: Fixed default robot properties (for test urdf generation)

File: srs_chuck/src/srsbot_chuck/urdf/config/robot_properties.xacro (robot description, xacro)
@@ -49,10 +49,6 @@
     <!-- Sensors -->
     <!-- Realsense -->
-    <xacro:property name="realsense_z_offset" value="-0.09766" />
-    <!-- Stargazer -->
-    <!-- All measurements made from base_link -> bottom left corner of stargazer -->
-    <xacro:property name="stargazer_x_offset" value="-0.4217162" />
-    <xacro:property name="stargazer_y_offset" value="-0.0352552" />
-    <xacro:property name="stargazer_z_offset" value="0.998982" />
+    <xacro:property name="realsense_z_rotation" value="${M_PI}" />
+    <xacro:property name="realsense_z_offset" value="0.0641858" />
     <!-- SICK Lidar -->
     <xacro:property name="lidar_x_offset" value="0.4600448" />
